File: hardware/canbus_connector.kicad_sch (KiCad schematic)
At the start: 2 parts

Commit message: Added analog stage for Vbat measurement, and it's simulation
Connections:
- net GND: now also J201.9 (SH), J202.9 (SH); no longer J201.SH, J202.SH
Changed lines of the file:
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@@
     (pin "1")
   )
-  (symbol (lib_id "Connector:RJ45_Shielded") (at 177.8 72.39 0) (mirror y) (unit 1)
+  (symbol (lib_name "RJ45_Shielded_1") (lib_id "Connector:RJ45_Shielded") (at 177.8 72.39 0) (mirror y) (unit 1)
     (in_bom yes) (on_board yes)
-    (property "Reference" "J201" (id 0) (at 172.72 58.42 0))
-    (property "Value" "~" (id 1) (at 181.61 58.42 0))
+    (property "Reference" "J201" (id 0) (at 182.88 58.42 0))
+    (property "Value" "~" (id 1) (at 173.99 58.42 0))
     (property "Footprint" "KicadZeniteSolarLibrary18:RJ45_YH59_01" (id 2) (at 177.8 72.39 0)
       (effects (font (size 1.27 1.27)) hide)
@@
     (pin "7")
     (pin "8")
-    (pin "SH")
+    (pin "9")
   )
   (symbol (lib_id "power:GND") (at 107.95 82.55 0) (unit 1)
@@
   (symbol (lib_id "Connector:RJ45_Shielded") (at 217.17 72.39 0) (mirror y) (unit 1)
     (in_bom yes) (on_board yes)
-    (property "Reference" "J202" (id 0) (at 212.09 58.42 0))
-    (property "Value" "~" (id 1) (at 220.98 58.42 0))
+    (property "Reference" "J202" (id 0) (at 222.25 58.42 0))
+    (property "Value" "~" (id 1) (at 213.36 58.42 0))
     (property "Footprint" "KicadZeniteSolarLibrary18:RJ45_YH59_01" (id 2) (at 217.17 72.39 0)
       (effects (font (size 1.27 1.27)) hide)
@@
     (pin "7")
     (pin "8")
-    (pin "SH")
+    (pin "9")
   )
 )
