File: hardware/canbus.kicad_sch (KiCad schematic)
At the start: 21 parts, among them U201 MCP2561-E/SN, U202 MCP2515-I/SO, Y402 16MHz

Commit message: Created BOM, removed Testpoints from it.
Parts:
- TP401, TP402, TP403, TP404, TP406, TP407, TP408, TP409: value TestPoint -> (none); footprint TestPoint:TestPoint_Pad_2.0x2.0mm -> (none); now left out of the parts list
Changed lines of the file:
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@@
   )
   (symbol (lib_id "Connector:TestPoint") (at 193.04 91.44 90) (unit 1)
-    (in_bom yes) (on_board yes) (fields_autoplaced)
+    (in_bom no) (on_board yes) (fields_autoplaced)
     (property "Reference" "TP408" (id 0) (at 189.738 87.1052 90))
-    (property "Value" "TestPoint" (id 1) (at 189.738 89.6421 90))
-    (property "Footprint" "TestPoint:TestPoint_Pad_2.0x2.0mm" (id 2) (at 193.04 86.36 0)
+    (property "Value" "" (id 1) (at 189.738 89.6421 90))
+    (property "Footprint" "" (id 2) (at 193.04 86.36 0)
       (effects (font (size 1.27 1.27)) hide)
     )
@@
   )
   (symbol (lib_id "Connector:TestPoint") (at 223.52 91.44 270) (unit 1)
-    (in_bom yes) (on_board yes) (fields_autoplaced)
+    (in_bom no) (on_board yes) (fields_autoplaced)
     (property "Reference" "TP409" (id 0) (at 228.219 90.6053 90)
       (effects (font (size 1.27 1.27)) (justify left))
     )
-    (property "Value" "TestPoint" (id 1) (at 228.219 93.1422 90)
+    (property "Value" "" (id 1) (at 228.219 93.1422 90)
       (effects (font (size 1.27 1.27)) (justify left))
     )
-    (property "Footprint" "TestPoint:TestPoint_Pad_2.0x2.0mm" (id 2) (at 223.52 96.52 0)
+    (property "Footprint" "" (id 2) (at 223.52 96.52 0)
       (effects (font (size 1.27 1.27)) hide)
     )
@@
   )
   (symbol (lib_id "Connector:TestPoint") (at 78.74 90.17 180) (unit 1)
-    (in_bom yes) (on_board yes) (fields_autoplaced)
+    (in_bom no) (on_board yes) (fields_autoplaced)
     (property "Reference" "TP401" (id 0) (at 80.137 92.6373 0)
       (effects (font (size 1.27 1.27)) (justify right))
     )
-    (property "Value" "TestPoint" (id 1) (at 80.137 95.1742 0)
+    (property "Value" "" (id 1) (at 80.137 95.1742 0)
       (effects (font (size 1.27 1.27)) (justify right))
     )
-    (property "Footprint" "TestPoint:TestPoint_Pad_2.0x2.0mm" (id 2) (at 73.66 90.17 0)
+    (property "Footprint" "" (id 2) (at 73.66 90.17 0)
       (effects (font (size 1.27 1.27)) hide)
     )
@@
   )
   (symbol (lib_id "Connector:TestPoint") (at 82.55 87.63 180) (unit 1)
-    (in_bom yes) (on_board yes) (fields_autoplaced)
+    (in_bom no) (on_board yes) (fields_autoplaced)
     (property "Reference" "TP402" (id 0) (at 83.947 90.0973 0)
       (effects (font (size 1.27 1.27)) (justify right))
     )
-    (property "Value" "TestPoint" (id 1) (at 83.947 92.6342 0)
+    (property "Value" "" (id 1) (at 83.947 92.6342 0)
       (effects (font (size 1.27 1.27)) (justify right))
     )
-    (property "Footprint" "TestPoint:TestPoint_Pad_2.0x2.0mm" (id 2) (at 77.47 87.63 0)
+    (property "Footprint" "" (id 2) (at 77.47 87.63 0)
       (effects (font (size 1.27 1.27)) hide)
     )
@@
   )
   (symbol (lib_id "Connector:TestPoint") (at 140.97 82.55 180) (unit 1)
-    (in_bom yes) (on_board yes) (fields_autoplaced)
+    (in_bom no) (on_board yes) (fields_autoplaced)
     (property "Reference" "TP407" (id 0) (at 142.367 85.0173 0)
       (effects (font (size 1.27 1.27)) (justify right))
     )
-    (property "Value" "TestPoint" (id 1) (at 142.367 87.5542 0)
+    (property "Value" "" (id 1) (at 142.367 87.5542 0)
       (effects (font (size 1.27 1.27)) (justify right))
     )
-    (property "Footprint" "TestPoint:TestPoint_Pad_2.0x2.0mm" (id 2) (at 135.89 82.55 0)
+    (property "Footprint" "" (id 2) (at 135.89 82.55 0)
       (effects (font (size 1.27 1.27)) hide)
     )
@@
   )
   (symbol (lib_id "Connector:TestPoint") (at 90.17 76.2 0) (unit 1)
-    (in_bom yes) (on_board yes) (fields_autoplaced)
+    (in_bom no) (on_board yes) (fields_autoplaced)
     (property "Reference" "TP404" (id 0) (at 91.567 72.0633 0)
       (effects (font (size 1.27 1.27)) (justify left))
     )
-    (property "Value" "TestPoint" (id 1) (at 91.567 74.6002 0)
+    (property "Value" "" (id 1) (at 91.567 74.6002 0)
       (effects (font (size 1.27 1.27)) (justify left))
     )
-    (property "Footprint" "TestPoint:TestPoint_Pad_2.0x2.0mm" (id 2) (at 95.25 76.2 0)
+    (property "Footprint" "" (id 2) (at 95.25 76.2 0)
       (effects (font (size 1.27 1.27)) hide)
     )
@@
   )
   (symbol (lib_id "Connector:TestPoint") (at 86.36 77.47 0) (unit 1)
-    (in_bom yes) (on_board yes) (fields_autoplaced)
+    (in_bom no) (on_board yes) (fields_autoplaced)
     (property "Reference" "TP403" (id 0) (at 87.757 73.3333 0)
       (effects (font (size 1.27 1.27)) (justify left))
     )
-    (property "Value" "TestPoint" (id 1) (at 87.757 75.8702 0)
+    (property "Value" "" (id 1) (at 87.757 75.8702 0)
       (effects (font (size 1.27 1.27)) (justify left))
     )
-    (property "Footprint" "TestPoint:TestPoint_Pad_2.0x2.0mm" (id 2) (at 91.44 77.47 0)
+    (property "Footprint" "" (id 2) (at 91.44 77.47 0)
       (effects (font (size 1.27 1.27)) hide)
     )
@@
   )
   (symbol (lib_id "Connector:TestPoint") (at 140.97 77.47 0) (unit 1)
-    (in_bom yes) (on_board yes) (fields_autoplaced)
+    (in_bom no) (on_board yes) (fields_autoplaced)
     (property "Reference" "TP406" (id 0) (at 142.367 73.3333 0)
       (effects (font (size 1.27 1.27)) (justify left))
     )
-    (property "Value" "TestPoint" (id 1) (at 142.367 75.8702 0)
+    (property "Value" "" (id 1) (at 142.367 75.8702 0)
       (effects (font (size 1.27 1.27)) (justify left))
     )
-    (property "Footprint" "TestPoint:TestPoint_Pad_2.0x2.0mm" (id 2) (at 146.05 77.47 0)
+    (property "Footprint" "" (id 2) (at 146.05 77.47 0)
       (effects (font (size 1.27 1.27)) hide)
     )
